Commit message: [ADD] a home model

File: src/tinker_description/urdf/sensor/hokuyo_lx30_laser.urdf.xacro (robot description, xacro)
@@ -16,5 +16,5 @@
                 <geometry>
                     <!--box size=".04 .04 .05"/-->
-                    <mesh filename="package://tinker_description/src/meshes/hokuyo.dae"/>
+                    <mesh filename="package://tinker_description/meshes/hokuyo.dae"/>
                 </geometry>
             </visual>
