Commit message: laser fusion running

File: src/tinker_description/urdf/base/base.urdf.xacro (robot description, xacro)
@@ -13,5 +13,5 @@
     <xacro:property name="base_width" value="0.4"/>
     <xacro:property name="base_height" value="0.15"/>
-    <xacro:property name="base_laser_x" value="0.27"/>
+    <xacro:property name="base_laser_x" value="0"/>
     <xacro:property name="base_laser_y" value="0"/>
     <xacro:property name="base_laser_z" value="0.185"/>

Commit message: [Change] Tune navigation for release 2.1(HK Journalist)

File: src/tinker_description/urdf/base/base.urdf.xacro (robot description, xacro)
@@ -13,5 +13,5 @@
     <xacro:property name="base_width" value="0.4"/>
     <xacro:property name="base_height" value="0.15"/>
-    <xacro:property name="base_laser_x" value="0"/>
+    <xacro:property name="base_laser_x" value="0.27"/>
     <xacro:property name="base_laser_y" value="0"/>
     <xacro:property name="base_laser_z" value="0.185"/>

Commit message: [Fix] Prohibit moving backwards

File: src/tinker_description/urdf/base/base.urdf.xacro (robot description, xacro)
@@ -10,8 +10,8 @@
     <xacro:property name="PI" value="3.1415926535897931"/>
     <xacro:property name="base_mass" value="1"/>
-    <xacro:property name="base_length" value="0.6"/>
-    <xacro:property name="base_width" value="0.4"/>
+    <xacro:property name="base_length" value="0.64"/>
+    <xacro:property name="base_width" value="0.52"/>
     <xacro:property name="base_height" value="0.15"/>
-    <xacro:property name="base_laser_x" value="0.27"/>
+    <xacro:property name="base_laser_x" value="0.30"/>
     <xacro:property name="base_laser_y" value="0"/>
     <xacro:property name="base_laser_z" value="0.185"/>

Commit message: [Add] kinect & arm urdf

File: src/tinker_description/urdf/base/base.urdf.xacro (robot description, xacro)
@@ -16,4 +16,10 @@
     <xacro:property name="base_laser_y" value="0"/>
     <xacro:property name="base_laser_z" value="0.185"/>
+    <xacro:property name="kinect_x" value="0"/>
+    <xacro:property name="kinect_y" value="0.20"/>
+    <xacro:property name="kinect_z" value="1.26"/>
+    <xacro:property name="arm_origin_x" value="0.12"/>
+    <xacro:property name="arm_origin_y" value="0"/>
+    <xacro:property name="arm_origin_z" value="0.77"/>
     <xacro:property name="wheel_mass" value="1"/>
 <!--*****************chasiss***********************-->
@@ -45,3 +51,16 @@
       <origin xyz="${base_laser_x} ${base_laser_y} ${base_laser_z}" rpy="0 0 0" />
   </xacro:hokuyo_lx30_laser_v0>
+<!--*****************base_to_arm_platform***********************-->
+    <link name="kinect_link" />
+    <link name="arm_link" />
+    <joint name="kinect_joint" type="fixed">
+        <parent link="base_link" />
+        <child link="kinect_link" />
+        <origin xyz="${kinect_x} ${kinect_y} ${kinect_z}" rpy="0 0 0" />
+    </joint>
+    <joint name="arm_origin_joint" type="fixed">
+        <parent link="base_link" />
+        <child link="arm_link" />
+        <origin xyz="${arm_origin_x} ${arm_origin_y} ${arm_origin_z}" rpy="0 0 0" />
+    </joint>
 </robot>
